File: PCB/SCHEMATICS/SCHEMATICS.kicad_pcb (KiCad board)
At the start: 2 copper layers, 100 x 100 mm, 100 parts, among them IC1 CP2102-GMR, J1 Conn_01x24_Pin, J2 Conn_01x24_Pin, Q1 PMOS, U1 C7433, U3 LTR-303ALS-01, U5 LTR-303ALS-01, U6 C6482, U7 C6482

Commit message: Labeled modules
Parts:
- R40: value 510k -> Value: Value: Value: Value: Value: Value: 510k
Connections:
- TP25 pad : Net-(U6-VCC) -> (no net)
Other:
- board text added: "3V3 Reg"
- board text added: "B Sens"
- board text added: "Battery Charging"
- board text added: "Battery Level LEDS"
- board text added: "Design Men Group 09 Ankush (CHHANK001) Murray (INGMURO02) Tinashe (TMBTIN004)"
- board text added: "EPROM"
- board text added: "EPROM Spare"
- board text added: "Light Sensor"
- board text added: "Spare Reg"
- board text added: "Spare Sensor"
- board text added: "USB Module"
- board text added: "UVLO :)"
Changed lines of the file:
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@@
         (effects (font (size 1 1) (thickness 0.15)))
     )
-    (fp_text value "510k" (at 0 1.98) (layer "F.Fab")
+    (fp_text value "Value: Value: Value: Value: Value: Value:  510k" (at 0 1.98) (layer "F.Fab") hide
         (effects (font (size 1 1) (thickness 0.15)))
     )
@@
     (fp_circle (center 0 0) (end 1.5 0)
       (stroke (width 0.05) (type solid)) (fill none) (layer "F.CrtYd"))
-    (pad "" smd circle (at 0 0 180) (size 2 2) (layers "F.Cu")
-      (net 16 "Net-(U6-VCC)"))
+    (pad "" smd circle (at 0 0 180) (size 2 2) (layers "F.Cu"))
   )
   (footprint "footprint:RESC1005X40N" (layer "F.Cu")
@@
     (fp_arc (start 1.080188 -0.709627) (mid 1.299286 -0.618875) (end 1.390018 -0.399772)
       (stroke (width 0.254) (type solid)) (layer "F.SilkS"))
-    (fp_arc (start 1.390018 0.400203) (mid 1.299267 0.619284) (end 1.080188 0.710033)
+    (fp_arc (start 1.390018 0.400203) (mid 1.299267 0.61928) (end 1.080188 0.710033)
       (stroke (width 0.254) (type solid)) (layer "F.SilkS"))
     (fp_circle (center -0.800102 0.400051) (end -0.77013 0.400051)
@@
     (property "Sheetfile" "MICROCONTROLLER.kicad_sch")
     (property "Sheetname" "MICROCONTROLLER")
+    (property "dnp" "")
+    (property "exclude_from_bom" "")
     (property "ki_description" "Generic connector, single row, 01x24, script generated")
     (property "ki_keywords" "connector")
-    (attr through_hole)
+    (attr through_hole exclude_from_bom)
     (fp_text reference "J2" (at 0 -2.77 90) (layer "F.SilkS")
         (effects (font (size 1 1) (thickness 0.15)))
@@
     (property "Sheetfile" "POWER_MODULE.kicad_sch")
     (property "Sheetname" "POWER MODULE")
-    (attr smd)
+    (property "dnp" "")
+    (property "exclude_from_bom" "")
+    (attr smd exclude_from_bom)
     (fp_text reference "U9" (at 0 -0.5 unlocked) (layer "F.SilkS")
         (effects (font (size 1 1) (thickness 0.15)))
@@
     (property "Sheetfile" "MICROCONTROLLER.kicad_sch")
     (property "Sheetname" "MICROCONTROLLER")
+    (property "dnp" "")
+    (property "exclude_from_bom" "")
     (property "ki_description" "Generic connector, single row, 01x24, script generated")
     (property "ki_keywords" "connector")
-    (attr through_hole)
+    (attr through_hole exclude_from_bom)
     (fp_text reference "J1" (at 0 -2.77 90) (layer "F.SilkS")
         (effects (font (size 1 1) (thickness 0.15)))
@@
   (gr_rect (start 90 48) (end 190 148)
     (stroke (width 0.1) (type default)) (fill none) (layer "Edge.Cuts"))
+  (gr_text "3V3 Reg" (at 96 95) (layer "F.SilkS")
+    (effects (font (size 1 1) (thickness 0.2) bold) (justify left bottom))
+  )
+  (gr_text "EPROM Spare" (at 172 132) (layer "F.SilkS")
+    (effects (font (size 1 1) (thickness 0.2) bold) (justify left bottom))
+  )
+  (gr_text "Light Sensor" (at 92 138) (layer "F.SilkS")
+    (effects (font (size 1 1) (thickness 0.2) bold) (justify left bottom))
+  )
+  (gr_text "Design Men \nGroup 09\nAnkush (CHHANK001)\nMurray (INGMURO02)\nTinashe (TMBTIN004)" (at 176 145) (layer "F.SilkS")
+    (effects (font (size 1 0.8) (thickness 0.2) bold) (justify left bottom))
+  )
+  (gr_text "Battery Level LEDS" (at 154 99 90) (layer "F.SilkS")
+    (effects (font (size 0.6 0.6) (thickness 0.15) bold) (justify left bottom))
+  )
+  (gr_text "Spare Sensor " (at 124 145) (layer "F.SilkS")
+    (effects (font (size 1 1) (thickness 0.2) bold) (justify left bottom))
+  )
+  (gr_text "EPROM" (at 147 145) (layer "F.SilkS")
+    (effects (font (size 1 1) (thickness 0.2) bold) (justify left bottom))
+  )
+  (gr_text "USB Module" (at 105 72) (layer "F.SilkS")
+    (effects (font (size 1 1) (thickness 0.2) bold) (justify left bottom))
+  )
+  (gr_text "Spare Reg" (at 175 89) (layer "F.SilkS")
+    (effects (font (size 1 1) (thickness 0.2) bold) (justify left bottom))
+  )
+  (gr_text "Battery Charging " (at 138 88 90) (layer "F.SilkS")
+    (effects (font (size 1 1) (thickness 0.2) bold) (justify left bottom))
+  )
+  (gr_text "B Sens" (at 161 74) (layer "F.SilkS")
+    (effects (font (size 1 1) (thickness 0.2) bold) (justify left bottom))
+  )
+  (gr_text "UVLO :)" (at 175 76) (layer "F.SilkS")
+    (effects (font (size 1 1) (thickness 0.2) bold) (justify left bottom))
+  )
   (segment (start 112.422008 135.612033) (end 112.422008 135.204008) (width 0.25) (layer "F.Cu") (net 1))
   (segment (start 112.422008 141.808008) (end 112.422008 135.612033) (width 0.25) (layer "F.Cu") (net 1))
