File: PCB/SCHEMATICS/SENSING.kicad_sch (KiCad schematic)
At the start: 22 parts, among them U3 LTR-303ALS-01, U5 LTR-303ALS-01

Commit message: Updated pcb
Parts:
- added TP16, TP17, TP36: TestPoint, TestPoint:TestPoint_Pad_D2.0mm, symbol Connector:TestPoint
Connections:
- net GND: no longer C5.1, U5.3 (GND), U5.5 (INT)
- new net: TP36.1, U5.3 (GND)
- new net: C5.1, TP16.1
- new net: TP17.1, U5.5 (INT)
Changed lines of the file:
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@@
     (effects (font (size 1.27 1.27)) (justify left))
   )
+  (symbol (lib_id "Connector:TestPoint") (at 118.11 124.46 180) (unit 1)
+    (in_bom yes) (on_board yes) (dnp no) (fields_autoplaced)
+    (property "Reference" "TP36" (at 120.65 127.127 0)
+      (effects (font (size 1.27 1.27)) (justify right))
+    )
+    (property "Value" "TestPoint" (at 120.65 129.667 0)
+      (effects (font (size 1.27 1.27)) (justify right))
+    )
+    (property "Footprint" "TestPoint:TestPoint_Pad_D2.0mm" (at 113.03 124.46 0)
+      (effects (font (size 1.27 1.27)) hide)
+    )
+    (property "Datasheet" "~" (at 113.03 124.46 0)
+      (effects (font (size 1.27 1.27)) hide)
+    )
+    (pin "1")
+    (instances
+      (project "SCHEMATICS"
+        (path "/c9ca3a5c-30cb-4dce-b611-3270b9f3284b/1428f64b-a76f-4ab8-8617-b5b39829c481"
+          (reference "TP36") (unit 1)
+        )
+      )
+    )
+  )
   (symbol (lib_id "Device:C") (at 109.22 100.33 90) (unit 1)
     (in_bom yes) (on_board yes) (dnp no) (fields_autoplaced)
@@
     )
   )
-  (symbol (lib_id "power:GND") (at 134.62 118.11 0) (unit 1)
-    (in_bom yes) (on_board yes) (dnp no) (fields_autoplaced)
-    (property "Reference" "#PWR022" (at 134.62 124.46 0)
-      (effects (font (size 1.27 1.27)) hide)
-    )
-    (property "Value" "GND" (at 134.62 122.2455 0)
-      (effects (font (size 1.27 1.27)))
-    )
-    (property "Footprint" "" (at 134.62 118.11 0)
-      (effects (font (size 1.27 1.27)) hide)
-    )
-    (property "Datasheet" "" (at 134.62 118.11 0)
-      (effects (font (size 1.27 1.27)) hide)
-    )
-    (pin "1")
-    (instances
-      (project "SCHEMATICS"
-        (path "/c9ca3a5c-30cb-4dce-b611-3270b9f3284b/1428f64b-a76f-4ab8-8617-b5b39829c481"
-          (reference "#PWR022") (unit 1)
-        )
-      )
-    )
-  )
   (symbol (lib_id "Device:R_Small_US") (at 60.96 57.15 0) (unit 1)
     (in_bom yes) (on_board yes) (dnp no) (fields_autoplaced)
@@
         (path "/c9ca3a5c-30cb-4dce-b611-3270b9f3284b/1428f64b-a76f-4ab8-8617-b5b39829c481"
           (reference "R20") (unit 1)
-        )
-      )
-    )
-  )
-  (symbol (lib_id "power:GND") (at 101.6 100.33 270) (unit 1)
-    (in_bom yes) (on_board yes) (dnp no) (fields_autoplaced)
-    (property "Reference" "#PWR020" (at 95.25 100.33 0)
-      (effects (font (size 1.27 1.27)) hide)
-    )
-    (property "Value" "GND" (at 97.79 100.965 90)
-      (effects (font (size 1.27 1.27)) (justify right))
-    )
-    (property "Footprint" "" (at 101.6 100.33 0)
-      (effects (font (size 1.27 1.27)) hide)
-    )
-    (property "Datasheet" "" (at 101.6 100.33 0)
-      (effects (font (size 1.27 1.27)) hide)
-    )
-    (pin "1")
-    (instances
-      (project "SCHEMATICS"
-        (path "/c9ca3a5c-30cb-4dce-b611-3270b9f3284b/1428f64b-a76f-4ab8-8617-b5b39829c481"
-          (reference "#PWR020") (unit 1)
         )
       )
@@
     )
   )
+  (symbol (lib_id "Connector:TestPoint") (at 101.6 100.33 90) (unit 1)
+    (in_bom yes) (on_board yes) (dnp no) (fields_autoplaced)
+    (property "Reference" "TP16" (at 98.298 95.25 90)
+      (effects (font (size 1.27 1.27)))
+    )
+    (property "Value" "TestPoint" (at 98.298 97.79 90)
+      (effects (font (size 1.27 1.27)))
+    )
+    (property "Footprint" "TestPoint:TestPoint_Pad_D2.0mm" (at 101.6 95.25 0)
+      (effects (font (size 1.27 1.27)) hide)
+    )
+    (property "Datasheet" "~" (at 101.6 95.25 0)
+      (effects (font (size 1.27 1.27)) hide)
+    )
+    (pin "1")
+    (instances
+      (project "SCHEMATICS"
+        (path "/c9ca3a5c-30cb-4dce-b611-3270b9f3284b/1428f64b-a76f-4ab8-8617-b5b39829c481"
+          (reference "TP16") (unit 1)
+        )
+      )
+    )
+  )
   (symbol (lib_id "Connector:TestPoint") (at 55.88 40.64 0) (unit 1)
     (in_bom yes) (on_board yes) (dnp no)
@@
     )
   )
-  (symbol (lib_id "power:GND") (at 118.11 124.46 0) (unit 1)
-    (in_bom yes) (on_board yes) (dnp no) (fields_autoplaced)
-    (property "Reference" "#PWR021" (at 118.11 130.81 0)
-      (effects (font (size 1.27 1.27)) hide)
-    )
-    (property "Value" "GND" (at 118.11 129.54 0)
-      (effects (font (size 1.27 1.27)))
-    )
-    (property "Footprint" "" (at 118.11 124.46 0)
-      (effects (font (size 1.27 1.27)) hide)
-    )
-    (property "Datasheet" "" (at 118.11 124.46 0)
-      (effects (font (size 1.27 1.27)) hide)
-    )
-    (pin "1")
-    (instances
-      (project "SCHEMATICS"
-        (path "/c9ca3a5c-30cb-4dce-b611-3270b9f3284b/1428f64b-a76f-4ab8-8617-b5b39829c481"
-          (reference "#PWR021") (unit 1)
-        )
-      )
-    )
-  )
   (symbol (lib_id "power:GND") (at 195.58 72.39 0) (unit 1)
     (in_bom yes) (on_board yes) (dnp no) (fields_autoplaced)
@@
         )
       )
+    )
+  )
+  (symbol (lib_id "Connector:TestPoint") (at 134.62 118.11 180) (unit 1)
+    (in_bom yes) (on_board yes) (dnp no) (fields_autoplaced)
+    (property "Reference" "TP17" (at 137.16 120.777 0)
+      (effects (font (size 1.27 1.27)) (justify right))
+    )
+    (property "Value" "TestPoint" (at 137.16 123.317 0)
+      (effects (font (size 1.27 1.27)) (justify right))
+    )
+    (property "Footprint" "TestPoint:TestPoint_Pad_D2.0mm" (at 129.54 118.11 0)
+      (effects (font (size 1.27 1.27)) hide)
+    )
+    (property "Datasheet" "~" (at 129.54 118.11 0)
+      (effects (font (size 1.27 1.27)) hide)
+    )
+    (pin "1")
+    (instances
+      (project "SCHEMATICS"
+        (path "/c9ca3a5c-30cb-4dce-b611-3270b9f3284b/1428f64b-a76f-4ab8-8617-b5b39829c481"
+          (reference "TP17") (unit 1)
+        )
+      )
