File: PCB/SCHEMATICS/POWER_MODULE.kicad_sch (KiCad schematic)
At the start: 44 parts, among them Q1 PMOS, U1 C7433, U2 AMS1117-3.3, U4 AMS1117-3.3

Commit message: Updated pcb
Parts:
- removed U2, U4: AMS1117-3.3, footprint:SOT-223-4_L6.5-W3.5-P2.30-LS7.0-BR, symbol Regulator_Linear:AMS1117-3.3
- added REF1, REF2: AMS1117-3_3_C369933, footprint:SOT-223-4_L6.5-W3.5-P2.30-LS7.0-BR, symbol ams:AMS1117-3_3_C369933
- R40: value Value: Value: 510k -> Value: Value: Value: Value: 510k
- TP11, TP12, TP28, TP29: PART  TP8 -> (none)
Connections:
- net GND: now also REF1.1 (GND/ADJ); no longer C3.1, D2.2 (A), R7.1, TP29.1, TP6.1, TP8.1
- net at TP28.1: now also REF2.2 (Output)
- net at C2.1, D2.1 (K), D4.C (K)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: now also REF1.3 (Input)
- net at TP11.1: now also REF2.4 (Output)
- net at TP12.1: now also REF2.1 (GND/ADJ)
- new net: C3.1, D2.2 (A), R7.1, REF1.4 (Output), TP6.1, TP8.1
- new net: REF2.3 (Input), TP29.1
- no-connect marks 0 -> 1
Other:
- moved on the sheet: TP8

Commit message: Made changes
Parts:
- R40: value Value: Value: Value: Value: 510k -> Value: Value: Value: Value: Value: 510k
Changed lines of the file:
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@@
       (effects (font (size 1.27 1.27)) (justify left))
     )
-    (property "Value" "Value: Value: Value: Value:  510k" (at 174.625 139.7 0) (show_name)
+    (property "Value" "Value: Value: Value: Value: Value:  510k" (at 174.625 139.7 0) (show_name)
       (effects (font (size 1.27 1.27)) (justify left))
     )

Commit message: Labeled modules
Parts:
- U9: now not fitted; now left out of the parts list
Changed lines of the file:
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@@
   )
   (symbol (lib_id "Battery:18650") (at 59.055 140.335 0) (unit 1)
-    (in_bom yes) (on_board yes) (dnp no) (fields_autoplaced)
+    (in_bom no) (on_board yes) (dnp yes) (fields_autoplaced)
     (property "Reference" "U9" (at 60.325 140.335 0)
       (effects (font (size 1.27 1.27)))

Commit message: Justins reccomendations
Parts:
- removed D5: D_Schottky, footprint:SOT323_INFINEON, symbol Device:D_Schottky
Connections:
- net at Q1.3 (S), R10.2, R11.2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: now also R15.2
Changed lines of the file:
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@@
-    (stroke (width 0) (type default))
-  )
-  (wire (pts (xy 156.845 140.97) (xy 157.48 140.97))
     (stroke (width 0) (type default))
   )
@@
     (stroke (width 0) (type default))
   )
-  (wire (pts (xy 142.24 140.97) (xy 149.225 140.97))
+  (wire (pts (xy 142.24 140.97) (xy 157.48 140.97))
     (stroke (width 0) (type default))
   )
@@
         )
       )
-    )
-  )
-  (symbol (lib_name "D_Schottky_1") (lib_id "Device:D_Schottky") (at 153.035 140.97 180) (unit 1)
-    (in_bom yes) (on_board yes) (dnp no) (fields_autoplaced)
-    (property "Reference" "D5" (at 152.7175 145.2499 0)
-      (effects (font (size 1.27 1.27)))
-    )
-    (property "Value" "D_Schottky" (at 152.7175 143.3289 0)
-      (effects (font (size 1.27 1.27)))
-    )
-    (property "Footprint" "footprint:SOT323_INFINEON" (at 153.035 138.43 0)
-      (effects (font (size 1.27 1.27)) hide)
-    )
-    (property "Datasheet" "~" (at 153.035 148.59 0)
-      (effects (font (size 1.27 1.27)) hide)
-    )
-    (property "Extended" "" (at 153.035 140.97 0)
-      (effects (font (size 1.27 1.27)) hide)
-    )
-    (property "Total" "" (at 153.035 140.97 0)
-      (effects (font (size 1.27 1.27)) hide)
-    )
-    (property "Unit Price" "0.0167" (at 153.035 146.05 0)
-      (effects (font (size 1.27 1.27)) hide)
-    )
-    (property "PART " "    C191023" (at 155.575 148.59 0)
-      (effects (font (size 1.27 1.27)) hide)
-    )
-    (pin "A")
-    (pin "C")
-    (instances
-      (project "SCHEMATICS"
-        (path "/c9ca3a5c-30cb-4dce-b611-3270b9f3284b/c574ee02-103d-4bad-a8c0-5ec1707f609e"
-          (reference "D5") (unit 1)
-        )
-      )
